Commit message: necessary changes for vtr3 development

File: grizzly_description/urdf/add_frame.urdf.xacro (robot description, xacro)
@@ -33,32 +33,32 @@
        xmlns:xacro="http://ros.org/wiki/xacro"
        name="grizzly_tf">
-  <property name="x_com"
+  <xacro:property name="x_com"
             value="0.00000000" />
   <!-- com : center of mass -->
-  <property name="y_com"
+  <xacro:property name="y_com"
             value="0.00000000" />
   <!-- com : center of mass -->
-  <property name="z_com"
+  <xacro:property name="z_com"
             value="0.00000000" />
   <!-- com : center of mass -->
-  <property name="mass"
+  <xacro:property name="mass"
             value="0.1" />
   <!-- in kg-->
-  <property name="ixx_com_cs"
+  <xacro:property name="ixx_com_cs"
             value="0.01" />
   <!-- at center of mass aligned with coordinate system, kg*m^2-->
-  <property name="ixy_com_cs"
+  <xacro:property name="ixy_com_cs"
             value="0.0" />
   <!-- at center of mass aligned with coordinate system, kg*m^2-->
-  <property name="ixz_com_cs"
+  <xacro:property name="ixz_com_cs"
             value="0.0" />
   <!-- at center of mass aligned with coordinate system, kg*m^2-->
-  <property name="iyy_com_cs"
+  <xacro:property name="iyy_com_cs"
             value="0.01" />
   <!-- at center of mass aligned with coordinate system, kg*m^2-->
-  <property name="iyz_com_cs"
+  <xacro:property name="iyz_com_cs"
             value="0.00" />
   <!-- at center of mass aligned with coordinate system, kg*m^2-->
-  <property name="izz_com_cs"
+  <xacro:property name="izz_com_cs"
             value="0.01" />
   <!-- at center of mass aligned with coordinate system, kg*m^2-->

File: grizzly_description/urdf/base.urdf.xacro (robot description, xacro)
@@ -46,50 +46,50 @@
   <!-- PROPERTY LIST -->
   <!--All units in m-kg-s-radians unit system -->
-  <property name="M_PI"
+  <xacro:property name="M_PI"
             value="3.1415926535897931" />
   <!-- Main Body-base-->
   <!-- Location of com : center of mass -->
-  <property name="base_x_com"
+  <xacro:property name="base_x_com"
             value="-0.08748000" />
-  <property name="base_y_com"
+  <xacro:property name="base_y_com"
             value="-0.00085000" />
-  <property name="base_z_com"
+  <xacro:property name="base_z_com"
             value="0.09947000" />
   <!-- Size of the base-->
-  <property name="base_x_size"
+  <xacro:property name="base_x_size"
             value="0.708" />
-  <property name="base_y_size"
+  <xacro:property name="base_y_size"
             value="0.3" />
-  <property name="base_z_size"
+  <xacro:property name="base_z_size"
             value="1.826" />
   <!-- Mass of the base-->
-  <property name="base_mass" value="487" />
+  <xacro:property name="base_mass" value="487" />
   <!-- Mass of the front axle-->
-  <property name="front_axle_mass" value="113" />
+  <xacro:property name="front_axle_mass" value="113" />
   <!--Inertial values for the front_axle at center of mass, aligned with coordinate system. Units are kg*m^2-->
-  <property name="front_axle_ixx_com_cs"
+  <xacro:property name="front_axle_ixx_com_cs"
             value="0.60216370" />
-  <property name="front_axle_ixy_com_cs"
+  <xacro:property name="front_axle_ixy_com_cs"
             value="-0.02364198" />
-  <property name="front_axle_ixz_com_cs"
+  <xacro:property name="front_axle_ixz_com_cs"
             value="-0.11972132" />
-  <property name="front_axle_iyy_com_cs"
+  <xacro:property name="front_axle_iyy_com_cs"
             value="1.73859574" />
-  <property name="front_axle_iyz_com_cs"
+  <xacro:property name="front_axle_iyz_com_cs"
             value="-0.00154437" />
-  <property name="front_axle_izz_com_cs"
+  <xacro:property name="front_axle_izz_com_cs"
             value="2.02955229" />
   <!--Inertial values for the base at center of mass, aligned with coordinate system. Units are kg*m^2-->
-  <property name="base_ixx_com_cs"
+  <xacro:property name="base_ixx_com_cs"
             value="0.60216370" />
-  <property name="base_ixy_com_cs"
+  <xacro:property name="base_ixy_com_cs"
             value="-0.02364198" />
-  <property name="base_ixz_com_cs"
+  <xacro:property name="base_ixz_com_cs"
             value="-0.11972132" />
-  <property name="base_iyy_com_cs"
+  <xacro:property name="base_iyy_com_cs"
             value="1.73859574" />
-  <property name="base_iyz_com_cs"
+  <xacro:property name="base_iyz_com_cs"
             value="-0.00154437" />
-  <property name="base_izz_com_cs"
+  <xacro:property name="base_izz_com_cs"
             value="2.02955229" />
   <!-- BASE-FOOTPRINT -->
@@ -144,14 +144,14 @@
   </gazebo>
   <!-- Add a sensor anchor link that points to the center of the robot top plate -->
-  <grizzly_tf parent="base_link" name="sensor_anchor_link"
+  <xacro:grizzly_tf parent="base_link" name="sensor_anchor_link"
     translateX="0" translateY="0" translateZ="0.45"
     rotateX="0.0" rotateY="0.0" rotateZ="0.0"/>
   <!-- Add a sensor anchor link for the imu -->
-  <grizzly_tf parent="sensor_anchor_link" name="imu_link"
+  <xacro:grizzly_tf parent="sensor_anchor_link" name="imu_link"
     translateX="-0.788" translateY="0" translateZ="-0.118"
     rotateX="3.1415" rotateY="1.5701" rotateZ="0" />
   <!-- DECORATIONS -->
   <!-- Bumpers -->
-  <grizzly_part parent="base_footprint"
+  <xacro:grizzly_part parent="base_footprint"
                 name="bumper"
                 mesh="bumper"
@@ -167,5 +167,5 @@
   </gazebo>
   <!-- Back wheels -->
-  <grizzly_wheel fb="back"
+  <xacro:grizzly_wheel fb="back"
                  lr="left"
                  parent="base_link"
@@ -174,5 +174,5 @@
                  translateZ="0"
                  flipY="0" />
-  <grizzly_wheel fb="back"
+  <xacro:grizzly_wheel fb="back"
                  lr="right"
                  parent="base_link"
@@ -228,5 +228,5 @@
   </gazebo>
   <!-- Front wheels -->
-  <grizzly_wheel fb="front"
+  <xacro:grizzly_wheel fb="front"
                  lr="left"
                  parent="front_axle_link"
@@ -235,5 +235,5 @@
                  translateZ="0"
                  flipY="0" />
-  <grizzly_wheel fb="front"
+  <xacro:grizzly_wheel fb="front"
                  lr="right"
                  parent="front_axle_link"

File: grizzly_description/urdf/parts.urdf.xacro (robot description, xacro)
@@ -33,38 +33,38 @@
        xmlns:xacro="http://ros.org/wiki/xacro"
        name="grizzly_part">
-  <property name="x_com"
+  <xacro:property name="x_com"
             value="0.00000000" />
   <!-- com : center of mass -->
-  <property name="y_com"
+  <xacro:property name="y_com"
             value="0.00000000" />
   <!-- com : center of mass -->
-  <property name="z_com"
+  <xacro:property name="z_com"
             value="0.00000000" />
   <!-- com : center of mass -->
-  <property name="x_size"
+  <xacro:property name="x_size"
             value="1.0" />
-  <property name="y_size"
+  <xacro:property name="y_size"
             value="1.0" />
-  <property name="z_size"
+  <xacro:property name="z_size"
             value="1.0" />
-  <property name="mass"
+  <xacro:property name="mass"
             value="0.1" />
   <!-- in kg-->
-  <property name="ixx_com_cs"
+  <xacro:property name="ixx_com_cs"
             value="0.01" />
   <!-- at center of mass aligned with coordinate system, kg*m^2-->
-  <property name="ixy_com_cs"
+  <xacro:property name="ixy_com_cs"
             value="0.0" />
   <!-- at center of mass aligned with coordinate system, kg*m^2-->
-  <property name="ixz_com_cs"
+  <xacro:property name="ixz_com_cs"
             value="0.0" />
   <!-- at center of mass aligned with coordinate system, kg*m^2-->
-  <property name="iyy_com_cs"
+  <xacro:property name="iyy_com_cs"
             value="0.01" />
   <!-- at center of mass aligned with coordinate system, kg*m^2-->
-  <property name="iyz_com_cs"
+  <xacro:property name="iyz_com_cs"
             value="0.00" />
   <!-- at center of mass aligned with coordinate system, kg*m^2-->
-  <property name="izz_com_cs"
+  <xacro:property name="izz_com_cs"
             value="0.01" />
   <!-- at center of mass aligned with coordinate system, kg*m^2-->

File: grizzly_description/urdf/wheel.urdf.xacro (robot description, xacro)
@@ -30,48 +30,48 @@
        xmlns:xacro="http://ros.org/wiki/xacro"
        name="grizzly_wheel">
-  <property name="M_PI"
+  <xacro:property name="M_PI"
             value="3.14159" />
   <!-- Wheel -->
-  <property name="wheel_x_com"
+  <xacro:property name="wheel_x_com"
             value="0.00000000" />
   <!-- com : center of mass -->
-  <property name="wheel_y_com"
+  <xacro:property name="wheel_y_com"
             value="0.00000000" />
   <!-- com : center of mass -->
-  <property name="wheel_z_com"
+  <xacro:property name="wheel_z_com"
             value="0.00019000" />
   <!-- com : center of mass -->
-  <property name="wheel_x_size"
+  <xacro:property name="wheel_x_size"
             value="0.66" />
-  <property name="wheel_y_size"
+  <xacro:property name="wheel_y_size"
             value="0.66" />
-  <property name="wheel_z_size"
+  <xacro:property name="wheel_z_size"
             value="0.252" />
-  <property name="wheel_mass" value="15" />
-  <property name="wheel_ixx_com_cs"
+  <xacro:property name="wheel_mass" value="15" />
+  <xacro:property name="wheel_ixx_com_cs"
             value="0.02466885" />
   <!-- at center of mass aligned with coordinate system, kg*m^2-->
-  <property name="wheel_ixy_com_cs"
+  <xacro:property name="wheel_ixy_com_cs"
             value="0.00000000" />
   <!-- at center of mass aligned with coordinate system, kg*m^2-->
-  <property name="wheel_ixz_com_cs"
+  <xacro:property name="wheel_ixz_com_cs"
             value="0.00000000" />
   <!-- at center of mass aligned with coordinate system, kg*m^2-->
-  <property name="wheel_iyy_com_cs"
+  <xacro:property name="wheel_iyy_com_cs"
             value="0.02466885" />
   <!-- at center of mass aligned with coordinate system, kg*m^2-->
-  <property name="wheel_iyz_com_cs"
+  <xacro:property name="wheel_iyz_com_cs"
             value="0.00000000" />
   <!-- at center of mass aligned with coordinate system, kg*m^2-->
-  <property name="wheel_izz_com_cs"
+  <xacro:property name="wheel_izz_com_cs"
             value="0.04410576" />
   <!-- at center of mass aligned with coordinate system, kg*m^2-->
-  <property name="base_x_origin_to_wheel_origin"
+  <xacro:property name="base_x_origin_to_wheel_origin"
             value="0.25600006" />
-  <property name="base_y_origin_to_wheel_origin"
+  <xacro:property name="base_y_origin_to_wheel_origin"
             value="0.285475" />
-  <property name="base_z_origin_to_wheel_origin"
+  <xacro:property name="base_z_origin_to_wheel_origin"
             value="0.0" />
-  <property name="base_z_origin_offset"
+  <xacro:property name="base_z_origin_offset"
             value="0.2" />
   <!-- origin is offset in + z direction by 3.175mm, so need to bring it back down for visual and collision-->
